Commit message: [up] changed the repo and project naming.

File: urdf/cr_hand_urdf.xacro (robot description, xacro)
@@ -1,7 +1,7 @@
 <?xml version="1.0" ?>
-<robot name="CR-Hand_URDF" xmlns:xacro="http://www.ros.org/wiki/xacro">
-<xacro:include filename="$(find CR-Hand_URDF)/urdf/materials.xacro" />
-<xacro:include filename="$(find CR-Hand_URDF)/urdf/sensors.xacro" />
-<xacro:include filename="$(find CR-Hand_URDF)/urdf/CR-Hand_URDF.gazebo" />
+<robot name="cr_hand_urdf" xmlns:xacro="http://www.ros.org/wiki/xacro">
+<xacro:include filename="$(find cr_hand_urdf)/urdf/materials.xacro" />
+<xacro:include filename="$(find cr_hand_urdf)/urdf/sensors.xacro" />
+<xacro:include filename="$(find cr_hand_urdf)/urdf/cr_hand_urdf.gazebo" />
 <link name="base_link">
   <inertial>
@@ -13,5 +13,5 @@
     <origin xyz="0 0 0" rpy="0 0 0"/>
     <geometry>
-      <mesh filename="file://$(find CR-Hand_URDF)/meshes/base_link.stl" scale="0.001 0.001 0.001"/>
+      <mesh filename="file://$(find cr_hand_urdf)/meshes/base_link.stl" scale="0.001 0.001 0.001"/>
     </geometry>
     <material name="silver"/>
@@ -20,5 +20,5 @@
     <origin xyz="0 0 0" rpy="0 0 0"/>
     <geometry>
-      <mesh filename="file://$(find CR-Hand_URDF)/meshes/base_link.stl" scale="0.001 0.001 0.001"/>
+      <mesh filename="file://$(find cr_hand_urdf)/meshes/base_link.stl" scale="0.001 0.001 0.001"/>
     </geometry>
   </collision>
@@ -33,5 +33,5 @@
     <origin xyz="-0.0225 -0.0255 -0.143" rpy="0 0 0"/>
     <geometry>
-      <mesh filename="file://$(find CR-Hand_URDF)/meshes/link2_2_1.stl" scale="0.001 0.001 0.001"/>
+      <mesh filename="file://$(find cr_hand_urdf)/meshes/link2_2_1.stl" scale="0.001 0.001 0.001"/>
     </geometry>
     <material name="silver"/>
@@ -40,5 +40,5 @@
     <origin xyz="-0.0225 -0.0255 -0.143" rpy="0 0 0"/>
     <geometry>
-      <mesh filename="file://$(find CR-Hand_URDF)/meshes/link2_2_1.stl" scale="0.001 0.001 0.001"/>
+      <mesh filename="file://$(find cr_hand_urdf)/meshes/link2_2_1.stl" scale="0.001 0.001 0.001"/>
     </geometry>
   </collision>
@@ -53,5 +53,5 @@
     <origin xyz="-0.0225 -0.0255 -0.103" rpy="0 0 0"/>
     <geometry>
-      <mesh filename="file://$(find CR-Hand_URDF)/meshes/link2_1_1.stl" scale="0.001 0.001 0.001"/>
+      <mesh filename="file://$(find cr_hand_urdf)/meshes/link2_1_1.stl" scale="0.001 0.001 0.001"/>
     </geometry>
     <material name="silver"/>
@@ -60,5 +60,5 @@
     <origin xyz="-0.0225 -0.0255 -0.103" rpy="0 0 0"/>
     <geometry>
-      <mesh filename="file://$(find CR-Hand_URDF)/meshes/link2_1_1.stl" scale="0.001 0.001 0.001"/>
+      <mesh filename="file://$(find cr_hand_urdf)/meshes/link2_1_1.stl" scale="0.001 0.001 0.001"/>
     </geometry>
   </collision>
@@ -73,5 +73,5 @@
     <origin xyz="-0.02255 -0.005028 -0.148439" rpy="0 0 0"/>
     <geometry>
-      <mesh filename="file://$(find CR-Hand_URDF)/meshes/link3_2_1.stl" scale="0.001 0.001 0.001"/>
+      <mesh filename="file://$(find cr_hand_urdf)/meshes/link3_2_1.stl" scale="0.001 0.001 0.001"/>
     </geometry>
     <material name="silver"/>
@@ -80,5 +80,5 @@
     <origin xyz="-0.02255 -0.005028 -0.148439" rpy="0 0 0"/>
     <geometry>
-      <mesh filename="file://$(find CR-Hand_URDF)/meshes/link3_2_1.stl" scale="0.001 0.001 0.001"/>
+      <mesh filename="file://$(find cr_hand_urdf)/meshes/link3_2_1.stl" scale="0.001 0.001 0.001"/>
     </geometry>
   </collision>
@@ -93,5 +93,5 @@
     <origin xyz="-0.02255 -0.006423 -0.108464" rpy="0 0 0"/>
     <geometry>
-      <mesh filename="file://$(find CR-Hand_URDF)/meshes/link3_1_1.stl" scale="0.001 0.001 0.001"/>
+      <mesh filename="file://$(find cr_hand_urdf)/meshes/link3_1_1.stl" scale="0.001 0.001 0.001"/>
     </geometry>
     <material name="silver"/>
@@ -100,5 +100,5 @@
     <origin xyz="-0.02255 -0.006423 -0.108464" rpy="0 0 0"/>
     <geometry>
-      <mesh filename="file://$(find CR-Hand_URDF)/meshes/link3_1_1.stl" scale="0.001 0.001 0.001"/>
+      <mesh filename="file://$(find cr_hand_urdf)/meshes/link3_1_1.stl" scale="0.001 0.001 0.001"/>
     </geometry>
   </collision>
@@ -113,5 +113,5 @@
     <origin xyz="-0.0225 0.015441 -0.144258" rpy="0 0 0"/>
     <geometry>
-      <mesh filename="file://$(find CR-Hand_URDF)/meshes/link4_2_1.stl" scale="0.001 0.001 0.001"/>
+      <mesh filename="file://$(find cr_hand_urdf)/meshes/link4_2_1.stl" scale="0.001 0.001 0.001"/>
     </geometry>
     <material name="silver"/>
@@ -120,5 +120,5 @@
     <origin xyz="-0.0225 0.015441 -0.144258" rpy="0 0 0"/>
     <geometry>
-      <mesh filename="file://$(find CR-Hand_URDF)/meshes/link4_2_1.stl" scale="0.001 0.001 0.001"/>
+      <mesh filename="file://$(find cr_hand_urdf)/meshes/link4_2_1.stl" scale="0.001 0.001 0.001"/>
     </geometry>
   </collision>
@@ -133,5 +133,5 @@
     <origin xyz="-0.0225 0.012651 -0.104355" rpy="0 0 0"/>
     <geometry>
-      <mesh filename="file://$(find CR-Hand_URDF)/meshes/link4_1_1.stl" scale="0.001 0.001 0.001"/>
+      <mesh filename="file://$(find cr_hand_urdf)/meshes/link4_1_1.stl" scale="0.001 0.001 0.001"/>
     </geometry>
     <material name="silver"/>
@@ -140,5 +140,5 @@
     <origin xyz="-0.0225 0.012651 -0.104355" rpy="0 0 0"/>
     <geometry>
-      <mesh filename="file://$(find CR-Hand_URDF)/meshes/link4_1_1.stl" scale="0.001 0.001 0.001"/>
+      <mesh filename="file://$(find cr_hand_urdf)/meshes/link4_1_1.stl" scale="0.001 0.001 0.001"/>
     </geometry>
   </collision>
@@ -153,5 +153,5 @@
     <origin xyz="-0.0225 0.035901 -0.139955" rpy="0 0 0"/>
     <geometry>
-      <mesh filename="file://$(find CR-Hand_URDF)/meshes/link5_2_1.stl" scale="0.001 0.001 0.001"/>
+      <mesh filename="file://$(find cr_hand_urdf)/meshes/link5_2_1.stl" scale="0.001 0.001 0.001"/>
     </geometry>
     <material name="silver"/>
@@ -160,5 +160,5 @@
     <origin xyz="-0.0225 0.035901 -0.139955" rpy="0 0 0"/>
     <geometry>
-      <mesh filename="file://$(find CR-Hand_URDF)/meshes/link5_2_1.stl" scale="0.001 0.001 0.001"/>
+      <mesh filename="file://$(find cr_hand_urdf)/meshes/link5_2_1.stl" scale="0.001 0.001 0.001"/>
     </geometry>
   </collision>
@@ -173,5 +173,5 @@
     <origin xyz="-0.0225 0.031719 -0.100174" rpy="0 0 0"/>
     <geometry>
-      <mesh filename="file://$(find CR-Hand_URDF)/meshes/link5_1_1.stl" scale="0.001 0.001 0.001"/>
+      <mesh filename="file://$(find cr_hand_urdf)/meshes/link5_1_1.stl" scale="0.001 0.001 0.001"/>
     </geometry>
     <material name="silver"/>
@@ -180,5 +180,5 @@
     <origin xyz="-0.0225 0.031719 -0.100174" rpy="0 0 0"/>
     <geometry>
-      <mesh filename="file://$(find CR-Hand_URDF)/meshes/link5_1_1.stl" scale="0.001 0.001 0.001"/>
+      <mesh filename="file://$(find cr_hand_urdf)/meshes/link5_1_1.stl" scale="0.001 0.001 0.001"/>
     </geometry>
   </collision>
@@ -193,5 +193,5 @@
     <origin xyz="-0.0225 -0.0545 -0.025" rpy="0 0 0"/>
     <geometry>
-      <mesh filename="file://$(find CR-Hand_URDF)/meshes/link1_3_1.stl" scale="0.001 0.001 0.001"/>
+      <mesh filename="file://$(find cr_hand_urdf)/meshes/link1_3_1.stl" scale="0.001 0.001 0.001"/>
     </geometry>
     <material name="silver"/>
@@ -200,5 +200,5 @@
     <origin xyz="-0.0225 -0.0545 -0.025" rpy="0 0 0"/>
     <geometry>
-      <mesh filename="file://$(find CR-Hand_URDF)/meshes/link1_3_1.stl" scale="0.001 0.001 0.001"/>
+      <mesh filename="file://$(find cr_hand_urdf)/meshes/link1_3_1.stl" scale="0.001 0.001 0.001"/>
     </geometry>
   </collision>
@@ -213,5 +213,5 @@
     <origin xyz="-0.0225 -0.0255 -0.028" rpy="0 0 0"/>
     <geometry>
-      <mesh filename="file://$(find CR-Hand_URDF)/meshes/link1_1_1.stl" scale="0.001 0.001 0.001"/>
+      <mesh filename="file://$(find cr_hand_urdf)/meshes/link1_1_1.stl" scale="0.001 0.001 0.001"/>
     </geometry>
     <material name="silver"/>
@@ -220,5 +220,5 @@
     <origin xyz="-0.0225 -0.0255 -0.028" rpy="0 0 0"/>
     <geometry>
-      <mesh filename="file://$(find CR-Hand_URDF)/meshes/link1_1_1.stl" scale="0.001 0.001 0.001"/>
+      <mesh filename="file://$(find cr_hand_urdf)/meshes/link1_1_1.stl" scale="0.001 0.001 0.001"/>
     </geometry>
   </collision>

File: urdf/materials.xacro (robot description, xacro)
@@ -1,6 +1,6 @@
-<?xml version="1.0" ?>
-<robot name="CR-Hand_URDF" xmlns:xacro="http://www.ros.org/wiki/xacro" >
-<material name="silver">
-  <color rgba="0.700 0.700 0.700 1.000"/>
-</material>
+<?xml version="1.0"?>
+<robot name="cr_hand_urdf" xmlns:xacro="http://www.ros.org/wiki/xacro">
+  <material name="silver">
+    <color rgba="0.700 0.700 0.700 1.000" />
+  </material>
 </robot>

File: urdf/sensors.xacro (robot description, xacro)
@@ -1,12 +1,12 @@
-<?xml version="1.0" ?>
-<robot name="CR-Hand_URDF" xmlns:xacro="http://www.ros.org/wiki/xacro" >
-<xacro:property name="yaml_file" value="$(find CR-Hand_URDF)/config/sensor_parameters.yaml" />
-<xacro:property name="params_dict" value="${xacro.load_yaml(yaml_file)}" />
-<xacro:property name="L2D_params" value="${params_dict['L2D']}" />
-<xacro:property name="L3D_params" value="${params_dict['L3D']}" />
-<xacro:property name="DCAM_params" value="${params_dict['DCAM']}" />
-<xacro:property name="CAM_params" value="${params_dict['CAM']}" />
-<xacro:property name="IMU_params" value="${params_dict['IMU']}" />
-<xacro:property name="GPS_params" value="${params_dict['GPS']}" />
-<xacro:property name="P3D_params" value="${params_dict['P3D']}" />
+<?xml version="1.0"?>
+<robot name="cr_hand_urdf" xmlns:xacro="http://www.ros.org/wiki/xacro">
+    <xacro:property name="yaml_file" value="$(find cr_hand_urdf)/config/sensor_parameters.yaml" />
+    <xacro:property name="params_dict" value="${xacro.load_yaml(yaml_file)}" />
+    <xacro:property name="L2D_params" value="${params_dict['L2D']}" />
+    <xacro:property name="L3D_params" value="${params_dict['L3D']}" />
+    <xacro:property name="DCAM_params" value="${params_dict['DCAM']}" />
+    <xacro:property name="CAM_params" value="${params_dict['CAM']}" />
+    <xacro:property name="IMU_params" value="${params_dict['IMU']}" />
+    <xacro:property name="GPS_params" value="${params_dict['GPS']}" />
+    <xacro:property name="P3D_params" value="${params_dict['P3D']}" />
 </robot>
